Commit message: Update IMU position

File: urdf/raspicat.urdf (robot description, URDF)
Before this commit: robot raspicat, 18 links, 17 joints
Joints:
- joint imu_joint: origin xyz=0 0 0.14 rpy=3.14 0 0 -> xyz=0 0 0.14 rpy=0 0 0

File: urdf/raspicat.urdf.xacro (robot description, xacro)
@@ -76,5 +76,5 @@
   <!-- Imu -->
   <xacro:imu_sensor prefix="imu" parent="base_link">
-    <origin xyz="0 0 0.14" rpy="${M_PI} 0 0"/>
+    <origin xyz="0 0 0.14" rpy="0 0 0"/>
   </xacro:imu_sensor>
   <!-- =============== Gazebo =============== -->

File: urdf/sensors/imu.gazebo.xacro (robot description, xacro)
@@ -52,4 +52,5 @@
             <remapping>~/out:=/${prefix}/data_raw</remapping>
           </ros>
+          <frame_name>base_link</frame_name>
         </plugin>
       </sensor>
